Commit message: model

File: src/gym_linefollower/envs/motoko_uprising.urdf (robot description, URDF)
Before this commit: robot line_follower, 10 links, 9 joints
Links:
- removed link front_left
- removed link front_right
- removed link main_board_0
- removed link main_board_1
- removed link main_board_left_a
- removed link main_board_left_b
- removed link main_board_right_a
- removed link main_board_right_b
- added link chassis, mass 0.063; collision mesh filename=./motoko_uprising.obj scale=0.001 0.001 0.001; visual mesh filename=./motoko_uprising.obj scale=0.001 0.001 0.001
Joints:
- removed joint main_board_0_left_wheel
- removed joint main_board_0_main_board_1
- removed joint main_board_0_main_board_left_a
- removed joint main_board_0_main_board_left_b
- removed joint main_board_0_main_board_right_a
- removed joint main_board_0_main_board_right_b
- removed joint main_board_0_right_wheel
- removed joint main_board_1_front_0
- removed joint main_board_1_front_1
- added joint chassis_left_wheel: type continuous, parent chassis, child left_wheel, origin xyz=-0.03 0.05 0.0025 rpy=-1.5708 0.0 0, axis 0 0 1
- added joint chassis_right_wheel: type continuous, parent chassis, child right_wheel, origin xyz=-0.03 -0.05 0.0025 rpy=1.5708 0.0 0, axis 0 0 -1
