Commit message: random lines added

File: src/gym_linefollower/envs/models/track_plane_template.urdf (robot description, URDF)
Before this commit: robot world, 2 links, 1 joints
Links:
- link line: geometry visual mesh filename=./models/track_plane_template.obj scale=1 1 1
- link plane: geometry collision box size=10.0 10.0 0.01; visual box size=10.0 10.0 0.001
